File: hardware/peripheral/p2sdc-001.brd (EAGLE design)
At the start: 91 x 90 mm, 6 parts, among them J2 GPIO, J5 SPI

Commit message: First try.
Parts:
- added R1: 10k, resistor:0204/5
- moved U$1 35.6 mm to (45.5, 38.0)
- moved LOGO1 23.6 mm to (45.5, 45.0)
Connections:
- net GND: now also JP1.3
- net GPIO0: now also JP1.7
- net GPIO1: now also JP1.8, R1.1
- net MISO: now also JP1.5
- net MOSI: now also JP1.6
- net SCK: now also JP1.4
- net VCC: now also JP1.1, R1.2
Routing:
- net VCC: track 0.00 -> 150.8 mm
- net GND: track 0.00 -> 150.4 mm
- net GPIO1: track 0.00 -> 68.7 mm
- net GPIO0: track 0.00 -> 43.3 mm
- net MOSI: track 0.00 -> 39.3 mm
- net MISO: track 0.00 -> 36.7 mm
- net SCK: track 0.00 -> 33.7 mm
Changed lines of the file:
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@@
 <setting verticaltext="up"/>
 </settings>
-<grid distance="1" unitdist="mm" unit="mm" style="lines" multiple="1" display="yes" altdistance="50" altunitdist="mil" altunit="mil"/>
+<grid distance="50" unitdist="mil" unit="mil" style="lines" multiple="2" display="yes" altdistance="50" altunitdist="mil" altunit="mil"/>
 <layers>
 <layer number="1" name="Top" color="4" fill="1" visible="yes" active="yes"/>
@@
 <wire x1="45.4" y1="58.25" x2="20" y2="58.25" width="0.15" layer="21"/>
 <wire x1="20" y1="58.25" x2="20" y2="90" width="0.15" layer="21"/>
-<hole x="22.54" y="87.46" drill="1"/>
-<hole x="42.86" y="87.46" drill="1"/>
-<hole x="22.54" y="64.6" drill="1"/>
-<hole x="42.86" y="64.6" drill="1"/>
+<hole x="22.54" y="87.46" drill="2.5"/>
+<hole x="42.86" y="87.46" drill="2.5"/>
+<hole x="22.54" y="64.6" drill="2.5"/>
+<hole x="42.86" y="64.6" drill="2.5"/>
+<text x="46.5" y="65" size="1" layer="25" align="center-left">4-M2.3</text>
+<circle x="22.54" y="87.46" radius="2" width="0.2" layer="42"/>
+<circle x="42.86" y="87.46" radius="2" width="0.2" layer="42"/>
+<circle x="42.86" y="64.6" radius="2" width="0.2" layer="42"/>
+<circle x="22.54" y="64.6" radius="2" width="0.2" layer="42"/>
+<circle x="22.54" y="87.46" radius="2" width="0.2" layer="41"/>
+<circle x="42.86" y="87.46" radius="2" width="0.2" layer="41"/>
+<circle x="22.54" y="64.6" radius="2" width="0.2" layer="41"/>
+<circle x="42.86" y="64.6" radius="2" width="0.2" layer="41"/>
 </plain>
 <attributes>
@@
 </autorouter>
 <elements>
-<element name="LOGO1" library="SparkFun-Aesthetics" package="OSHW-LOGO-S_COPPER" value="OSHW-LOGOS-COPPER" x="37" y="67" smashed="yes"/>
-<element name="U$1" library="pineapple" package="PINEAPPLE450_SILK" value="PINEAPPLE450_SILK" x="79" y="50" smashed="yes"/>
+<element name="LOGO1" library="SparkFun-Aesthetics" package="OSHW-LOGO-S_COPPER" value="OSHW-LOGOS-COPPER" x="45.5" y="45" smashed="yes"/>
+<element name="U$1" library="pineapple" package="PINEAPPLE450_SILK" value="PINEAPPLE450_SILK" x="45.5" y="38" smashed="yes"/>
 <element name="JP5" library="pinhead" library_urn="urn:adsk.eagle:library:325" package="1X03" package3d_urn="urn:adsk.eagle:package:22458/2" value="PWR" x="88" y="20" smashed="yes" rot="R90">
 <attribute name="NAME" x="85" y="20" size="1" layer="25" ratio="10" rot="R90" align="center"/>
@@
 <attribute name="VALUE" x="22.54" y="56.599" size="1.27" layer="27"/>
 </element>
+<element name="R1" library="resistor" library_urn="urn:adsk.eagle:library:348" package="0204/5" package3d_urn="urn:adsk.eagle:package:23488/1" value="10k" x="3" y="62" smashed="yes" rot="R90">
+<attribute name="NAME" x="1.8316" y="59.9934" size="0.9906" layer="25" ratio="10" rot="R90"/>
+<attribute name="VALUE" x="5.3114" y="59.8664" size="0.9906" layer="27" ratio="10" rot="R90"/>
+</element>
 </elements>
 <signals>
@@
 <contactref element="J2" pad="1"/>
 <contactref element="J5" pad="6"/>
-<wire x1="6" y1="31" x2="88" y2="17.46" width="0" layer="19" extent="1-1"/>
-<wire x1="3" y1="76.35" x2="6" y2="31" width="0" layer="19" extent="1-1"/>
+<contactref element="JP1" pad="3"/>
+<wire x1="7.62" y1="76.2762" x2="3.048" y2="76.2762" width="0.3048" layer="1"/>
+<wire x1="22.2504" y1="61.6458" x2="7.62" y2="76.2762" width="0.3048" layer="1"/>
+<wire x1="27.051" y1="61.6458" x2="24.9174" y2="61.6458" width="0.3048" layer="1"/>
+<wire x1="24.9174" y1="61.6458" x2="22.2504" y2="61.6458" width="0.3048" layer="1"/>
+<wire x1="28.8798" y1="59.817" x2="27.051" y2="61.6458" width="0.3048" layer="1"/>
+<wire x1="3.048" y1="76.2762" x2="3" y2="76.35" width="0.3048" layer="1"/>
+<wire x1="28.8798" y1="59.817" x2="28.89" y2="59.774" width="0.3048" layer="1"/>
+<wire x1="86.1822" y1="17.526" x2="87.9348" y2="17.526" width="0.3048" layer="1"/>
+<wire x1="42.0624" y1="61.6458" x2="86.1822" y2="17.526" width="0.3048" layer="1"/>
+<wire x1="30.861" y1="61.6458" x2="42.0624" y2="61.6458" width="0.3048" layer="1"/>
+<wire x1="29.0322" y1="59.817" x2="30.861" y2="61.6458" width="0.3048" layer="1"/>
+<wire x1="87.9348" y1="17.526" x2="88" y2="17.46" width="0.3048" layer="1"/>
+<wire x1="29.0322" y1="59.817" x2="28.89" y2="59.774" width="0.3048" layer="1"/>
+<wire x1="5.9436" y1="31.4706" x2="5.9436" y2="31.0134" width="0.3048" layer="1"/>
+<wire x1="4.8768" y1="32.5374" x2="5.9436" y2="31.4706" width="0.3048" layer="1"/>
+<wire x1="4.8768" y1="38.5572" x2="4.8768" y2="32.5374" width="0.3048" layer="1"/>
+<wire x1="24.9174" y1="58.5978" x2="4.8768" y2="38.5572" width="0.3048" layer="1"/>
+<wire x1="24.9174" y1="61.6458" x2="24.9174" y2="58.5978" width="0.3048" layer="1"/>
+<wire x1="5.9436" y1="31.0134" x2="6" y2="31" width="0.3048" layer="1"/>
 </signal>
 <signal name="VCC" class="2">
@@
 <contactref element="J2" pad="2"/>
 <contactref element="J5" pad="2"/>
-<wire x1="6" y1="33" x2="88" y2="20" width="0" layer="19" extent="1-1"/>
-<wire x1="3" y1="71.27" x2="6" y2="33" width="0" layer="19" extent="1-1"/>
+<contactref element="JP1" pad="1"/>
+<contactref element="R1" pad="2"/>
+<wire x1="3.9624" y1="70.3326" x2="3.048" y2="71.247" width="0.508" layer="1"/>
+<wire x1="3.9624" y1="65.4558" x2="3.9624" y2="70.3326" width="0.508" layer="1"/>
+<wire x1="3.048" y1="64.5414" x2="3.9624" y2="65.4558" width="0.508" layer="1"/>
+<wire x1="3.048" y1="71.247" x2="3" y2="71.27" width="0.508" layer="1"/>
+<wire x1="3.048" y1="64.5414" x2="3" y2="64.54" width="0.508" layer="1"/>
+<wire x1="9.7536" y1="59.817" x2="23.7744" y2="59.817" width="0.508" layer="1"/>
+<wire x1="4.191" y1="65.3796" x2="9.7536" y2="59.817" width="0.508" layer="1"/>
+<wire x1="23.7744" y1="59.817" x2="23.81" y2="59.774" width="0.508" layer="1"/>
+<wire x1="4.191" y1="65.3796" x2="3.9624" y2="65.4558" width="0.508" layer="1"/>
+<wire x1="18.9738" y1="20.0406" x2="87.9348" y2="20.0406" width="0.508" layer="16"/>
+<wire x1="6.0198" y1="32.9946" x2="18.9738" y2="20.0406" width="0.508" layer="16"/>
+<wire x1="87.9348" y1="20.0406" x2="88" y2="20" width="0.508" layer="16"/>
+<wire x1="6.0198" y1="32.9946" x2="6" y2="33" width="0.508" layer="16"/>
+<wire x1="2.9718" y1="60.96" x2="2.9718" y2="64.4652" width="0.508" layer="16"/>
+<wire x1="1.905" y1="59.8932" x2="2.9718" y2="60.96" width="0.508" layer="16"/>
+<wire x1="1.905" y1="37.0332" x2="1.905" y2="59.8932" width="0.508" layer="16"/>
+<wire x1="5.7912" y1="33.147" x2="1.905" y2="37.0332" width="0.508" layer="16"/>
+<wire x1="2.9718" y1="64.4652" x2="3" y2="64.54" width="0.508" layer="16"/>
+<wire x1="5.7912" y1="33.147" x2="6" y2="33" width="0.508" layer="16"/>
 </signal>
 <signal name="RST">
@@
 <signal name="GPIO1">
 <contactref element="J2" pad="4"/>
+<contactref element="JP1" pad="8"/>
+<contactref element="R1" pad="1"/>
+<wire x1="3.048" y1="39.9288" x2="3.048" y2="59.436" width="0.1524" layer="16"/>
+<wire x1="5.9436" y1="37.0332" x2="3.048" y2="39.9288" width="0.1524" layer="16"/>
+<wire x1="3.048" y1="59.436" x2="3" y2="59.46" width="0.1524" layer="16"/>
+<wire x1="5.9436" y1="37.0332" x2="6" y2="37" width="0.1524" layer="16"/>
+<wire x1="41.2242" y1="59.7408" x2="41.529" y2="59.7408" width="0.1524" layer="1"/>
+<wire x1="18.5166" y1="37.0332" x2="41.2242" y2="59.7408" width="0.1524" layer="1"/>
+<wire x1="6.0198" y1="37.0332" x2="18.5166" y2="37.0332" width="0.1524" layer="1"/>
+<wire x1="41.529" y1="59.7408" x2="41.59" y2="59.774" width="0.1524" layer="1"/>
+<wire x1="6.0198" y1="37.0332" x2="6" y2="37" width="0.1524" layer="1"/>
 </signal>
 <signal name="GPIO0">
 <contactref element="J2" pad="3"/>
+<contactref element="JP1" pad="7"/>
+<wire x1="38.7096" y1="59.7408" x2="39.0144" y2="59.7408" width="0.1524" layer="16"/>
+<wire x1="14.0208" y1="35.052" x2="38.7096" y2="59.7408" width="0.1524" layer="16"/>
+<wire x1="6.0198" y1="35.052" x2="14.0208" y2="35.052" width="0.1524" layer="16"/>
+<wire x1="39.0144" y1="59.7408" x2="39.05" y2="59.774" width="0.1524" layer="16"/>
+<wire x1="6.0198" y1="35.052" x2="6" y2="35" width="0.1524" layer="16"/>
 </signal>
 <signal name="V+" class="4">
@@
 <signal name="MISO">
 <contactref element="J5" pad="1"/>
+<contactref element="JP1" pad="5"/>
+<wire x1="11.43" y1="69.9516" x2="3.048" y2="69.9516" width="0.1524" layer="16"/>
+<wire x1="23.3934" y1="57.9882" x2="11.43" y2="69.9516" width="0.1524" layer="16"/>
+<wire x1="32.1564" y1="57.9882" x2="23.3934" y2="57.9882" width="0.1524" layer="16"/>
+<wire x1="33.909" y1="59.7408" x2="32.1564" y2="57.9882" width="0.1524" layer="16"/>
+<wire x1="3.048" y1="69.9516" x2="3" y2="70" width="0.1524" layer="16"/>
+<wire x1="33.909" y1="59.7408" x2="33.97" y2="59.774" width="0.1524" layer="16"/>
 </signal>
 <signal name="SCK">
 <contactref element="J5" pad="3"/>
+<contactref element="JP1" pad="4"/>
+<wire x1="18.7452" y1="72.4662" x2="3.048" y2="72.4662" width="0.1524" layer="16"/>
+<wire x1="31.3944" y1="59.817" x2="18.7452" y2="72.4662" width="0.1524" layer="16"/>
+<wire x1="3.048" y1="72.4662" x2="3" y2="72.54" width="0.1524" layer="16"/>
+<wire x1="31.3944" y1="59.817" x2="31.43" y2="59.774" width="0.1524" layer="16"/>
 </signal>
 <signal name="MOSI">
 <contactref element="J5" pad="4"/>
+<contactref element="JP1" pad="6"/>
+<wire x1="12.8016" y1="73.7616" x2="3.048" y2="73.7616" width="0.1524" layer="16"/>
+<wire x1="13.7922" y1="72.771" x2="12.8016" y2="73.7616" width="0.1524" layer="16"/>
+<wire x1="23.5458" y1="72.771" x2="13.7922" y2="72.771" width="0.1524" layer="16"/>
+<wire x1="36.4998" y1="59.817" x2="23.5458" y2="72.771" width="0.1524" layer="16"/>
+<wire x1="3.048" y1="73.7616" x2="3" y2="73.81" width="0.1524" layer="16"/>
+<wire x1="36.4998" y1="59.817" x2="36.51" y2="59.774" width="0.1524" layer="16"/>
 </signal>
 </signals>

Commit message: New interface.
Parts:
- removed J2: GPIO, SparkFun-Connectors:JST-4-PTH
- added J1: (no value), SparkFun-Connectors:1X04_1.27MM
- moved R1 4.00 mm to (3.00, 58.0)
Connections:
- net GND: no longer J2.1
- net GPIO0: now also J1.3; no longer J2.3
- net GPIO1: now also J1.4; no longer J2.4
- net VCC: no longer J2.2
Routing:
- net VCC: track 150.8 -> 115.7 mm
- net GND: track 150.4 -> 115.5 mm
- net GPIO1: track 68.7 -> 53.2 mm
- net GPIO0: track 43.3 -> 40.2 mm
- net SCK: track 33.7 -> 36.5 mm
- net MISO: track 36.7 -> 35.2 mm
- added copper zone on layer 1, net GND
- added copper zone on layer 16, net GND
Other:
- board text added: "0"
- board text added: "1"
- board text added: "N"
- board text added: "Pineapple IIb SD Card Adaptor 0.0.1-X"
- board text removed: "2.6.6-RC"
- board text removed: "G0"
- board text removed: "G1"
- board text removed: "GND"
- board text removed: "Pineapple IIb"
- board text removed: "RST"
